Commit message: Fixed Stop Sign and changed the PID and Pure Pursuit

File: src/gazebo_project/urdf/robot.urdf (robot description, URDF)
Before this commit: robot robot, 8 links, 7 joints
Links:
- link link_chassis: geometry collision box size=2.4 1.0 1.0; visual mesh filename=package://gazebo_project/meshes/smart_car.obj scale=0.012 0.012 0.013
